File: CKT-9000.brd (EAGLE design)
At the start: 25 x 25 mm, 8 parts, among them J1 PWR IN, J2 PWR OUT, J3 PI USB, J4 RX USB

Commit message: Adds a MOSFET and gate bias resistor to the board. The ID pin of the PWR IN usb connector is utilized as the signal to turn the MOSFET on/off.
Eagle Cad updated to v 9.5.1
Parts:
- added Q1: SI2342DS, brunnertech:SOT23
- added R1: 100K, brunnertech:R0805
- J2: value PWR OUT -> PI PWR
Connections:
- removed net ID$1: J1.ID, J2.ID
- removed net VBUS$2: J3.VBUS, J4.VBUS
- new net N$1: J3.VBUS, Q1.3
- new net N$2: J4.VBUS, Q1.2
- new net N$3: J1.ID, J2.ID, Q1.1, R1.2
- net GND: now also R1.1
Routing:
- net N$3: track 0.00 -> 21.6 mm
- net N$2: track 0.00 -> 16.5 mm
- net N$1: track 0.00 -> 12.4 mm
- net VBUS$2: track 11.9 -> 0.00 mm, vias 1 -> 0
- net ID$1: track 11.1 -> 0.00 mm, vias 1 -> 0
Other:
- board text added: "PCB-9000 A"
- board text removed: "PCB-9000"
Changed lines of the file:
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@@
 <?xml version="1.0" encoding="utf-8"?>
 <!DOCTYPE eagle SYSTEM "eagle.dtd">
-<eagle version="9.4.2">
+<eagle version="9.5.1">
 <drawing>
 <settings>
@@
 <setting verticaltext="up"/>
 </settings>
-<grid distance="0.1" unitdist="mm" unit="mm" style="dots" multiple="1" display="yes" altdistance="0.05" altunitdist="mm" altunit="mm"/>
+<grid distance="1" unitdist="mm" unit="mm" style="dots" multiple="1" display="yes" altdistance="0.1" altunitdist="mm" altunit="mm"/>
 <layers>
 <layer number="1" name="Top" color="4" fill="1" visible="yes" active="yes"/>
@@
 <dimension x1="0" y1="25" x2="25" y2="25" x3="12.5" y3="31.7" textsize="1.778" layer="51" dtype="horizontal"/>
 <dimension x1="0" y1="25" x2="0" y2="0" x3="-5.5" y3="12.5" textsize="1.778" layer="51" dtype="vertical"/>
-<text x="22.9" y="22.4" size="1.016" layer="16" ratio="18" rot="MR0">PCB-9000</text>
+<text x="22.9" y="22.4" size="1.016" layer="16" ratio="18" rot="MR0">PCB-9000 A</text>
 <text x="22.8" y="19.9" size="1.016" layer="22" ratio="18" rot="MR0">CKT-9000</text>
 <polygon width="0.127" layer="22">
@@
 <attribute name="VALUE" x="5" y="20.2" size="0.8198" layer="26" ratio="18" rot="MR0" align="top-center"/>
 </element>
-<element name="J2" library="brunnertech" package="GCT_USB3150" value="PWR OUT" x="5" y="14.3" smashed="yes" rot="R180">
+<element name="J2" library="brunnertech" package="GCT_USB3150" value="PI PWR" x="5" y="14.3" smashed="yes" rot="R180">
 <attribute name="NAME" x="1.9" y="16.1" size="0.8128" layer="25" ratio="18" rot="R180" align="top-center"/>
 <attribute name="VALUE" x="5" y="11.2" size="0.8192" layer="26" ratio="18" rot="MR180" align="top-center"/>
@@
 <element name="FID3" library="brunnertech" package="FIDUCIAL_1MM" value="FIDUCIAL&quot;&quot;" x="11.1" y="23" smashed="yes">
 <attribute name="BOM" value="EXCLUDE" x="11.1" y="23" size="1.778" layer="27" display="off"/>
+</element>
+<element name="Q1" library="brunnertech" package="SOT23" value="SI2342DS" x="11.3" y="16.7" smashed="yes">
+<attribute name="NAME" x="11.295" y="19.405" size="0.8198" layer="25" ratio="18" align="bottom-center"/>
+<attribute name="VALUE" x="11.295" y="14.525" size="0.4164" layer="27" ratio="10" align="top-center"/>
+</element>
+<element name="R1" library="brunnertech" package="R0805" package3d_urn="urn:adsk.eagle:package:23553/2" value="100K" x="11.3" y="10.6" smashed="yes" rot="R90">
+<attribute name="NAME" x="9.716" y="10.157" size="0.8128" layer="25" ratio="18" rot="R180" align="top-center"/>
+<attribute name="SPICEPREFIX" value="R" x="11.3" y="10.6" size="1.778" layer="27" rot="R90" display="off"/>
+<attribute name="VALUE" x="12.376" y="11.205" size="0.4064" layer="27" ratio="10" rot="R270"/>
 </element>
 </elements>
@@
 <polygon width="0.127" layer="16" pour="cutout">
 <vertex x="23.7" y="21.7"/>
-<vertex x="15.2" y="21.7"/>
-<vertex x="15.2" y="24.2"/>
+<vertex x="13.9" y="21.7"/>
+<vertex x="13.9" y="24.2"/>
 <vertex x="23.7" y="24.2"/>
 </polygon>
@@
 <wire x1="23.24" y1="2.81" x2="23.1" y2="2.81" width="0.1524" layer="1"/>
 <wire x1="23.1" y1="2.81" x2="23.1" y2="2.9072" width="0.1524" layer="1"/>
-</signal>
-<signal name="ID$1">
-<contactref element="J1" pad="ID"/>
-<contactref element="J2" pad="ID"/>
-<wire x1="4.35" y1="14.62" x2="4.35" y2="17.65" width="0.1524" layer="1"/>
-<wire x1="4" y1="18" x2="4" y2="19" width="0.1524" layer="1"/>
-<via x="4" y="19" extent="1-16" drill="0.35"/>
-<wire x1="4.35" y1="17.65" x2="4" y2="18" width="0.1524" layer="1"/>
-<wire x1="6.5306" y1="19.2197875" x2="6.5306" y2="18.7802125" width="0.1524" layer="16"/>
-<wire x1="6.5306" y1="18.7802125" x2="6.2197875" y2="18.4694" width="0.1524" layer="16"/>
-<wire x1="6.2197875" y1="18.4694" x2="5.7802125" y2="18.4694" width="0.1524" layer="16"/>
-<wire x1="5.7802125" y1="18.4694" x2="5.2496125" y2="19" width="0.1524" layer="16"/>
-<wire x1="5.2496125" y1="19" x2="4" y2="19" width="0.1524" layer="16"/>
-<wire x1="5.65" y1="20.1003875" x2="6.5306" y2="19.2197875" width="0.1524" layer="16"/>
-<wire x1="5.65" y1="22.08" x2="5.65" y2="20.1003875" width="0.1524" layer="16"/>
+<contactref element="R1" pad="1"/>
 </signal>
 <signal name="D-$1">
@@
 <wire x1="7.3" y1="16.5" x2="7.3" y2="15.17" width="0.254" layer="16"/>
 </signal>
-<signal name="VBUS$2">
-<contactref element="J3" pad="VBUS"/>
-<contactref element="J4" pad="VBUS"/>
-<wire x1="20.365" y1="4" x2="20.415" y2="4.05" width="0.1524" layer="1"/>
-<wire x1="18.4081" y1="13.3366" x2="18.4081" y2="12.6634" width="0.254" layer="16"/>
-<wire x1="18.9" y1="13.97" x2="18.9" y2="13.8285" width="0.254" layer="16"/>
-<wire x1="18.9" y1="13.8285" x2="18.4081" y2="13.3366" width="0.254" layer="16"/>
-<wire x1="18.4081" y1="12.6634" x2="18.9" y2="12.1715" width="0.254" layer="16"/>
-<via x="18.9" y="4" extent="1-16" drill="0.35"/>
-<wire x1="18.9" y1="4" x2="20.365" y2="4" width="0.254" layer="1"/>
-<wire x1="18.9" y1="12.1715" x2="18.9" y2="4" width="0.254" layer="16"/>
-</signal>
 <signal name="D+$2">
 <contactref element="J3" pad="D+"/>
@@
 <via x="16.95" y="6" extent="1-16" drill="0.35"/>
 <wire x1="16.95" y1="6" x2="20.415" y2="6" width="0.1524" layer="1"/>
+</signal>
+<signal name="N$1">
+<contactref element="J3" pad="VBUS"/>
+<contactref element="Q1" pad="3"/>
+<wire x1="11.3" y1="17.85" x2="18.6785" y2="17.85" width="0.254" layer="1"/>
+<wire x1="19.9919" y1="16.5366" x2="19.9919" y2="14.7634" width="0.254" layer="1"/>
+<wire x1="18.9" y1="13.97" x2="19.1985" y2="13.97" width="0.254" layer="1"/>
+<wire x1="19.9919" y1="14.7634" x2="19.1985" y2="13.97" width="0.254" layer="1"/>
+<wire x1="18.6785" y1="17.85" x2="19.9919" y2="16.5366" width="0.254" layer="1"/>
+</signal>
+<signal name="N$2">
+<contactref element="Q1" pad="2"/>
+<contactref element="J4" pad="VBUS"/>
+<wire x1="12.25" y1="15.8" x2="12.25" y2="13.75" width="0.254" layer="1"/>
+<wire x1="16.3686" y1="9.6314" x2="16.3686" y2="5.759175" width="0.254" layer="1"/>
+<wire x1="16.3686" y1="5.759175" x2="18.009175" y2="4.1186" width="0.254" layer="1"/>
+<wire x1="20.3464" y1="4.1186" x2="20.415" y2="4.05" width="0.254" layer="1"/>
+<wire x1="18.009175" y1="4.1186" x2="20.3464" y2="4.1186" width="0.254" layer="1"/>
+<wire x1="12.25" y1="13.75" x2="16.3686" y2="9.6314" width="0.254" layer="1"/>
+</signal>
+<signal name="N$3">
+<contactref element="J1" pad="ID"/>
+<contactref element="J2" pad="ID"/>
+<contactref element="Q1" pad="1"/>
+<contactref element="R1" pad="2"/>
+<wire x1="11.3" y1="11.55" x2="10.625" y2="12.225" width="0.1524" layer="1"/>
+<wire x1="10.625" y1="12.225" x2="10.35" y2="12.5" width="0.1524" layer="1"/>
+<wire x1="10.35" y1="12.5" x2="10.35" y2="15.8" width="0.1524" layer="1"/>
+<wire x1="5.65" y1="22.08" x2="5.9389" y2="21.7911" width="0.1524" layer="1"/>
+<wire x1="5.9389" y1="21.7911" x2="7.16555625" y2="21.7911" width="0.1524" layer="1"/>
+<wire x1="10.35" y1="15.8" x2="9.9767125" y2="15.8" width="0.1524" layer="1"/>
+<wire x1="9.9767125" y1="15.8" x2="8.6214" y2="17.1553125" width="0.1524" layer="1"/>
+<wire x1="7.16555625" y1="21.7911" x2="8.6214" y2="20.33525625" width="0.1524" layer="1"/>
+<wire x1="8.6214" y1="20.33525625" x2="8.6214" y2="17.1553125" width="0.1524" layer="1"/>
+<wire x1="4.35" y1="14.62" x2="4.3194" y2="14.5894" width="0.1524" layer="1"/>
+<wire x1="4.3194" y1="14.5894" x2="4.3194" y2="13.82950625" width="0.1524" layer="1"/>
+<wire x1="4.3194" y1="13.82950625" x2="5.92390625" y2="12.225" width="0.1524" layer="1"/>
+<wire x1="5.92390625" y1="12.225" x2="10.625" y2="12.225" width="0.1524" layer="1"/>
 </signal>
 </signals>
@@
 </board>
 </drawing>
+<compatibility>
+<note version="8.3" severity="warning">
+Since Version 8.3, EAGLE supports URNs for individual library
+assets (packages, symbols, and devices). The URNs of those assets
+will not be understood (or retained) with this version.
+</note>
+<note version="8.3" severity="warning">
+Since Version 8.3, EAGLE supports the association of 3D packages
+with devices in libraries, schematics, and board files. Those 3D
+packages will not be understood (or retained) with this version.
+</note>
+</compatibility>
 </eagle>

Commit message: Adds a second MOSFET (p-channel) along with an additional resistor to make the circuit actually do what it is supposed to. I obviously didn't think about the prior design very thoroughly! Here's the circuit I'm using to shoot for the correct behavior (with different FET's though): https://electronics.stackexchange.com/a/353222.  I also updated Eagle to the next minor release (9.5.2).
Parts:
- added Q2: SI2329DS, brunnertech:SOT23
- added R2: 100K, brunnertech:R0805
- moved R1 1.80 mm to (13.0, 10.0)
- moved Q1 1.60 mm to (11.3, 18.3), turned to 90 degrees
Connections:
- new net N$4: J4.VBUS, Q2.3
- net GND: now also Q1.2
- net N$1: now also Q2.1, R2.1; no longer J3.VBUS
- net N$2: now also J3.VBUS, Q2.2; no longer J4.VBUS, Q1.2
- net VBUS$1: now also R2.2
Routing:
- net N$4: track 0.00 -> 8.74 mm
- net N$3: track 21.6 -> 29.0 mm, vias 0 -> 1
- net VBUS$1: track 12.9 -> 19.1 mm
- net N$2: track 16.5 -> 18.4 mm, vias 0 -> 2
- net GND: track 11.3 -> 12.3 mm
- net N$1: track 12.4 -> 13.2 mm
Other:
- board text added: "PCB-9000 B"
- board text removed: "PCB-9000 A"
